File: MaxSingle.kicad_pcb (KiCad board)
At the start: 2 copper layers, 126 parts, among them J1 S2B-PH-K-S_LF__SN_, J2 OLED_128x64, SW1 1825910-6, SW2 RotaryEncoder, U2 nice_nano

Commit message: second changes
Parts:
- moved S61 135.9 mm to (80.6, 41.5), turned to 160 degrees
- moved SW1 130.2 mm to (344.6, 40.5), turned to 20 degrees
- moved J2 22.6 mm to (212.6, 148.1)
- moved SW2 21.8 mm to (215.1, 116.4), turned to -90 degrees
- moved U2 21.4 mm to (212.6, 96.5)
- moved D60 1.00 mm to (386.2, 125.5)
- moved D10 0.75 mm to (323.1, 63.9)
- moved D11 0.75 mm to (342.2, 60.7)
- moved D21 0.75 mm to (310.9, 86.0)
- moved D22 0.75 mm to (329.6, 81.8)
- moved D32 0.75 mm to (300.3, 112.7)
- moved D33 0.75 mm to (317.4, 104.0)
- moved D43 0.75 mm to (289.4, 138.2)
- moved D44 0.75 mm to (306.9, 130.6)
- moved D48 0.75 mm to (379.7, 107.9)
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